Commit message: changing the camera angle to have no pitch and simplifying perception algo

File: install/uuv_descriptions/share/uuv_descriptions/robots/generated/rexrov/robot_description.urdf (robot description, URDF)
Before this commit: robot rexrov, 26 links, 25 joints
Joints:
- joint rexrov/camera_joint: origin xyz=1.15 0 0.4 rpy=0 0.6 0 -> xyz=1.15 0 0.4 rpy=0 0 0
- joint rexrov/cameraleft_joint: origin xyz=1.15 0.63 0.4 rpy=0 0.6 -0.4 -> xyz=1.15 0.63 0.4 rpy=0 0 -0.4
- joint rexrov/cameraright_joint: origin xyz=1.15 -0.63 0.4 rpy=0 0.6 0.4 -> xyz=1.15 -0.63 0.4 rpy=0 0 0.4

File: install/uuv_descriptions/share/uuv_descriptions/urdf/rexrov_sensors.xacro (robot description, xacro)
@@ -44,11 +44,11 @@
   <!-- Mount a camera -->
   <xacro:default_camera namespace="${namespace}" parent_link="${namespace}/base_link" suffix="">
-    <origin xyz="1.15 0 0.4" rpy="0 0.6 0"/>
+    <origin xyz="1.15 0 0.4" rpy="0 0 0"/>
   </xacro:default_camera>
   <xacro:default_camera namespace="${namespace}" parent_link="${namespace}/base_link" suffix="right">
-    <origin xyz="1.15 -0.63 0.4" rpy="0 0.6 0.4"/>
+    <origin xyz="1.15 -0.63 0.4" rpy="0 0 0.4"/>
   </xacro:default_camera>
   <xacro:default_camera namespace="${namespace}" parent_link="${namespace}/base_link" suffix="left">
-    <origin xyz="1.15 0.63 0.4" rpy="0 0.6 -0.4"/>
+    <origin xyz="1.15 0.63 0.4" rpy="0 0 -0.4"/>
   </xacro:default_camera>
   <!-- Mount a GPS. -->
